Commit message: update sysID.

File: toddlerbot/descriptions/assemblies/使用长U支架_No_BATTERY_NO_CAP_SM40BL_sysID_assembly/使用长U支架_No_BATTERY_NO_CAP_SM40BL_sysID_assembly.urdf (robot description, URDF)
Before this commit: robot sysID_SM40BL, 2 links, 1 joints
Links:
- link sm40bl_mu_20190118: mass 0.544624 -> 0.236902

File: toddlerbot/descriptions/sysID_SM40BL/sysID_SM40BL.urdf (robot description, URDF)
Before this commit: robot sysID_SM40BL, 2 links, 1 joints
Links:
- link mount_sm40bl: geometry visual mesh filename=../assemblies/使用长U支架_No_BATTERY_NO_CAP_SM40BL_sysID_assembl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
- link sm40bl_mu_20190118: mass 0.544624 -> 0.236902; geometry visual mesh filename=../assemblies/使用长U支架_No_BATTERY_NO_CAP_SM40BL_sysID_assembl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
Joints:
- joint joint_0: limit lower=0 upper=3.14159 effort=10 velocity=10 -> lower=-1.5708 upper=1.5708 effort=10 velocity=10; origin xyz=0.0470055 0.0606694 0.0528278 rpy=0 -0 6.45317e-16 -> xyz=0.0470055 0.0647694 0.0722778 rpy=1.5708 -0 3.14159

File: toddlerbot/descriptions/sysID_SM40BL_2nd_backup/sysID_SM40BL.urdf (robot description, URDF)
Before this commit: robot sysID_SM40BL, 2 links, 1 joints
Links:
- link mount_sm40bl: geometry visual mesh filename=../assemblies/使用长U支架_SM40BL_sysID_assembly/meshes/mount_sm4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
- link sm40bl_mu_20190118: geometry visual mesh filename=../assemblies/使用长U支架_SM40BL_sysID_assembly/meshes/sm40bl_mu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
